File: PCB/PCB - alu40.brd (EAGLE design)
At the start: 228 x 76 mm, 163 parts, among them IC1 XB3303ASOT23, IC2 TP4054-42-SOT25-R, J1 SK-3296S-01-L1, J2 USB4510-03-1-A, Q2 PMOSFET, Q3 PMOSFET, Q5 PMOSFET, Q6 NMOSFET, U1 ISP1807-LRISP1807-LR_ISP1807-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, X1 BM02B-SRSS-TB

Commit message: Moved connector - added silk
Parts:
- moved X1 20.1 mm to (165.1, 59.8)
- moved C4 7.31 mm to (154.2, 57.7)
- moved R13 6.87 mm to (156.9, 56.5), turned to 0 degrees
- moved IC2 6.31 mm to (151.2, 58.3)
- moved R14 5.80 mm to (150.7, 61.1)
- moved IC1 5.31 mm to (146.2, 61.3)
- moved C5 5.20 mm to (146.3, 58.3)
- moved R15 5.20 mm to (146.3, 56.1)
- moved J4 5.10 mm to (142.4, 56.9)
- moved R17 4.88 mm to (159.2, 63.3)
Routing:
- net G_BAT: track 9.94 -> 30.2 mm, vias 0 -> 2
- net V_BATT: track 91.8 -> 111.5 mm, vias 2 -> 4
- net N$60: track 102.7 -> 109.0 mm
- net COL8: track 139.0 -> 135.1 mm
- net V_USB: track 240.0 -> 243.9 mm
- net N$53: track 5.55 -> 5.04 mm
- net GND: vias 19 -> 42
Other:
- board text added: "ALMN40 Rich Ying"

Commit message: Updated connector position
Parts:
- moved X1 0.22 mm to (165.0, 60.0), turned to 0 degrees
Routing:
- net V_BATT: track 111.5 -> 116.4 mm
Changed lines of the file:
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@@
 <element name="48-2" library="Volume_V1" library_urn="urn:adsk.eagle:library:32198814" package="CHERRY" package3d_urn="urn:adsk.eagle:package:32198958/1" value="" x="133" y="9.5" smashed="yes" rot="R180"/>
 <element name="46-2" library="Volume_V1" library_urn="urn:adsk.eagle:library:32198814" package="CHERRY" package3d_urn="urn:adsk.eagle:package:32198958/1" value="" x="114" y="9.5" smashed="yes" rot="R180"/>
-<element name="X1" library="Volume_V1" library_urn="urn:adsk.eagle:library:32198814" package="BM02B-SRSS-TB" package3d_urn="urn:adsk.eagle:package:32391209/2" value="BM02B-SRSS-TB" x="165.1" y="59.8" smashed="yes" rot="MR90">
-<attribute name="NAME" x="163.195" y="62.84" size="1.016" layer="26" rot="MR0" align="bottom-center"/>
-<attribute name="VALUE" x="166.37" y="60.3" size="1.016" layer="28" rot="MR90" align="bottom-right"/>
+<element name="X1" library="Volume_V1" library_urn="urn:adsk.eagle:library:32198814" package="BM02B-SRSS-TB" package3d_urn="urn:adsk.eagle:package:32391209/2" value="BM02B-SRSS-TB" x="165" y="60" smashed="yes" rot="MR0">
+<attribute name="NAME" x="161.96" y="58.095" size="1.016" layer="26" rot="MR270" align="bottom-center"/>
+<attribute name="VALUE" x="164.5" y="61.27" size="1.016" layer="28" rot="MR0" align="bottom-right"/>
 </element>
 <element name="Q3" library="Transistor" library_urn="urn:adsk.eagle:library:16378713" package="SOT23" package3d_urn="urn:adsk.eagle:package:28738/2" value="PMOSFET" x="143.5" y="40" smashed="yes" rot="MR180">
@@
 <wire x1="166.3" y1="54.8" x2="166.7" y2="54.8" width="0.508" layer="16"/>
 <via x="166.7" y="54.8" extent="1-16" drill="0.35"/>
-<wire x1="166.7" y1="54.8" x2="165.35" y2="56.15" width="0.508" layer="1"/>
+<wire x1="166.7" y1="54.8" x2="165.5" y2="56" width="0.508" layer="1"/>
 <wire x1="166.0572" y1="55.0428" x2="166.3" y2="54.8" width="0.508" layer="16"/>
-<wire x1="165.1" y1="59.3" x2="165.1" y2="58.1" width="0.508" layer="16"/>
-<wire x1="165.1" y1="58.1" x2="165.2" y2="58" width="0.508" layer="16"/>
-<via x="165.2" y="58" extent="1-16" drill="0.35"/>
-<wire x1="165.2" y1="58" x2="165.2" y2="56.3" width="0.508" layer="1"/>
-<wire x1="165.2" y1="56.3" x2="165.35" y2="56.15" width="0.508" layer="1"/>
+<wire x1="165.5" y1="61.9" x2="165.7" y2="62.1" width="0.508" layer="1"/>
+<via x="165.7" y="62.1" extent="1-16" drill="0.35"/>
+<wire x1="165.7" y1="62.1" x2="165.5" y2="61.9" width="0.508" layer="16"/>
+<wire x1="165.5" y1="61.9" x2="165.5" y2="60" width="0.508" layer="16"/>
+<wire x1="165.5" y1="56" x2="165.5" y2="61.9" width="0.508" layer="1"/>
 </signal>
 <signal name="G_BAT">
@@
 <wire x1="147.8" y1="61.3" x2="149.6" y2="63.1" width="0.508" layer="16"/>
 <wire x1="149.6" y1="63.1" x2="152.9" y2="63.1" width="0.508" layer="16"/>
-<wire x1="165.1" y1="60.3" x2="165.1" y2="61.6" width="0.508" layer="16"/>
-<wire x1="165.1" y1="61.6" x2="165" y2="61.7" width="0.508" layer="16"/>
-<via x="165" y="61.7" extent="1-16" drill="0.35"/>
-<wire x1="165" y1="61.7" x2="164.3" y2="62.4" width="0.508" layer="1"/>
-<wire x1="164.3" y1="62.4" x2="154.7" y2="62.4" width="0.508" layer="1"/>
+<wire x1="164.2" y1="62.1" x2="163.9" y2="62.4" width="0.508" layer="1"/>
+<wire x1="163.9" y1="62.4" x2="154.7" y2="62.4" width="0.508" layer="1"/>
+<wire x1="164.5" y1="61.8" x2="164.5" y2="60" width="0.508" layer="16"/>
+<wire x1="164.5" y1="61.8" x2="164.2" y2="62.1" width="0.508" layer="16"/>
+<via x="164.2" y="62.1" extent="1-16" drill="0.35"/>
 </signal>
 <signal name="BVOLT">

Commit message: Final connector update
Parts:
- moved X1 1.61 mm to (166.6, 59.8), turned to 90 degrees
Routing:
- net V_BATT: track 116.4 -> 111.3 mm
- net G_BAT: track 30.0 -> 33.2 mm
Changed lines of the file:
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@@
 <element name="48-2" library="Volume_V1" library_urn="urn:adsk.eagle:library:32198814" package="CHERRY" package3d_urn="urn:adsk.eagle:package:32198958/1" value="" x="133" y="9.5" smashed="yes" rot="R180"/>
 <element name="46-2" library="Volume_V1" library_urn="urn:adsk.eagle:library:32198814" package="CHERRY" package3d_urn="urn:adsk.eagle:package:32198958/1" value="" x="114" y="9.5" smashed="yes" rot="R180"/>
-<element name="X1" library="Volume_V1" library_urn="urn:adsk.eagle:library:32198814" package="BM02B-SRSS-TB" package3d_urn="urn:adsk.eagle:package:32391209/2" value="BM02B-SRSS-TB" x="165" y="60" smashed="yes" rot="MR0">
-<attribute name="NAME" x="161.96" y="58.095" size="1.016" layer="26" rot="MR270" align="bottom-center"/>
-<attribute name="VALUE" x="164.5" y="61.27" size="1.016" layer="28" rot="MR0" align="bottom-right"/>
+<element name="X1" library="Volume_V1" library_urn="urn:adsk.eagle:library:32198814" package="BM02B-SRSS-TB" package3d_urn="urn:adsk.eagle:package:32391209/2" value="BM02B-SRSS-TB" x="166.6" y="59.8" smashed="yes" rot="MR90">
+<attribute name="NAME" x="164.695" y="62.84" size="1.016" layer="26" rot="MR0" align="bottom-center"/>
+<attribute name="VALUE" x="167.87" y="60.3" size="1.016" layer="28" rot="MR90" align="bottom-right"/>
 </element>
 <element name="Q3" library="Transistor" library_urn="urn:adsk.eagle:library:16378713" package="SOT23" package3d_urn="urn:adsk.eagle:package:28738/2" value="PMOSFET" x="143.5" y="40" smashed="yes" rot="MR180">
@@
 <wire x1="166.3" y1="54.8" x2="166.7" y2="54.8" width="0.508" layer="16"/>
 <via x="166.7" y="54.8" extent="1-16" drill="0.35"/>
-<wire x1="166.7" y1="54.8" x2="165.5" y2="56" width="0.508" layer="1"/>
 <wire x1="166.0572" y1="55.0428" x2="166.3" y2="54.8" width="0.508" layer="16"/>
-<wire x1="165.5" y1="61.9" x2="165.7" y2="62.1" width="0.508" layer="1"/>
-<via x="165.7" y="62.1" extent="1-16" drill="0.35"/>
-<wire x1="165.7" y1="62.1" x2="165.5" y2="61.9" width="0.508" layer="16"/>
-<wire x1="165.5" y1="61.9" x2="165.5" y2="60" width="0.508" layer="16"/>
-<wire x1="165.5" y1="56" x2="165.5" y2="61.9" width="0.508" layer="1"/>
+<wire x1="166.7" y1="54.8" x2="167.2" y2="55.3" width="0.508" layer="1"/>
+<wire x1="167.2" y1="55.3" x2="167.2" y2="57.2" width="0.508" layer="1"/>
+<via x="167.2" y="57.2" extent="1-16" drill="0.35"/>
+<wire x1="166.6" y1="59.3" x2="166.6" y2="57.8" width="0.508" layer="16"/>
+<wire x1="167.2" y1="57.2" x2="166.6" y2="57.8" width="0.508" layer="16"/>
 </signal>
 <signal name="G_BAT">
@@
 <wire x1="154.1" y1="61.9" x2="152.9" y2="63.1" width="0.508" layer="16"/>
 <via x="154.1" y="61.8" extent="1-16" drill="0.35"/>
-<wire x1="154.7" y1="62.4" x2="154.1" y2="61.8" width="0.508" layer="1"/>
+<wire x1="154.1" y1="61.8" x2="154.7" y2="62.4" width="0.508" layer="1"/>
 <wire x1="147.8" y1="61.3" x2="149.6" y2="63.1" width="0.508" layer="16"/>
 <wire x1="149.6" y1="63.1" x2="152.9" y2="63.1" width="0.508" layer="16"/>
-<wire x1="164.2" y1="62.1" x2="163.9" y2="62.4" width="0.508" layer="1"/>
-<wire x1="163.9" y1="62.4" x2="154.7" y2="62.4" width="0.508" layer="1"/>
-<wire x1="164.5" y1="61.8" x2="164.5" y2="60" width="0.508" layer="16"/>
-<wire x1="164.5" y1="61.8" x2="164.2" y2="62.1" width="0.508" layer="16"/>
-<via x="164.2" y="62.1" extent="1-16" drill="0.35"/>
+<wire x1="166.9" y1="62.4" x2="167.6" y2="61.7" width="0.508" layer="1"/>
+<via x="167.6" y="61.7" extent="1-16" drill="0.35"/>
+<wire x1="166.6" y1="60.3" x2="166.6" y2="60.7" width="0.508" layer="16"/>
+<wire x1="167.6" y1="61.7" x2="166.6" y2="60.7" width="0.508" layer="16"/>
+<wire x1="154.7" y1="62.4" x2="166.9" y2="62.4" width="0.508" layer="1"/>
 </signal>
 <signal name="BVOLT">
