File: PCB/PCB - alu40.brd (EAGLE design)
At the start: 228 x 76 mm, 167 parts, among them IC1 XB3303ASOT23, IC2 TP4054-42-SOT25-R, J1 SK-3296S-01-L1, J2 USB4510-03-1-A, Q2 PMOSFET, Q3 PMOSFET, Q5 PMOSFET, Q6 NMOSFET, U1 ISP1807-LRISP1807-LR_ISP1807-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, X1 BM02B-SRSS-TB

Commit message: Change component vals
Parts:
- LED1: value (none) -> RED
- R14: value 200 -> 1.2k
Changed lines of the file:
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@@
 <drawing>
 <settings>
-<setting alwaysvectorfont="yes"/>
+<setting alwaysvectorfont="no"/>
 <setting verticaltext="up"/>
 </settings>
@@
 <attribute name="VALUE" x="157.535" y="54.595" size="1.27" layer="28" rot="MR0"/>
 </element>
-<element name="R14" library="rcl" library_urn="urn:adsk.eagle:library:334" package="R0603" package3d_urn="urn:adsk.eagle:package:23555/3" value="200" x="150.7" y="61.1" smashed="yes" rot="MR0">
+<element name="R14" library="rcl" library_urn="urn:adsk.eagle:library:334" package="R0603" package3d_urn="urn:adsk.eagle:package:23555/3" value="1.2k" x="150.7" y="61.1" smashed="yes" rot="MR0">
 <attribute name="NAME" x="151.335" y="61.735" size="1.27" layer="26" rot="MR0"/>
 <attribute name="POPULARITY" value="70" x="169.115" y="93.0024" size="1.778" layer="28" rot="MR0" display="off"/>
@@
 <attribute name="VALUE" x="84.881" y="72.849" size="0.6096" layer="28" font="vector" ratio="20" rot="MR0"/>
 </element>
-<element name="LED1" library="adafruit" library_urn="urn:adsk.eagle:library:420" package="CHIPLED_0805" package3d_urn="urn:adsk.eagle:package:6240559/1" value="" x="112" y="20" smashed="yes" rot="MR90">
+<element name="LED1" library="adafruit" library_urn="urn:adsk.eagle:library:420" package="CHIPLED_0805" package3d_urn="urn:adsk.eagle:package:6240559/1" value="RED" x="112" y="20" smashed="yes" rot="MR90">
 <attribute name="NAME" x="110.73" y="18.73" size="1.27" layer="26" rot="MR180"/>
 <attribute name="VALUE" x="110.73" y="22.54" size="1.27" layer="28" rot="MR180"/>
